File: eaglecad/modular_expansion_basic_joystick_only.sch (EAGLE design)
At the start: 31 parts, among them IC10 74ALS00N, IC11 74ALS00N, IC4 74ALS30N, IC6 74LS00N, IC7 74LS244N, IC8 7805TV, J1 JOY1, J3 POWERJACK

Commit message: various fixes
Changed lines of the file:
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@@
 <wire x1="55.88" y1="71.12" x2="55.88" y2="66.04" width="0.1524" layer="91"/>
 <junction x="55.88" y="71.12"/>
+<label x="0" y="71.12" size="1.778" layer="95"/>
 </segment>
 </net>
