File: eaglecad/modular_expansion_system_audio_mixer.brd (EAGLE design)
At the start: 81.6 x 100.2 mm, 82 parts, among them IC1 TL084P, J1 RCA, J1_ADDRESS_CON j1, J2 RCA, J2_DATA_AND_POWER_CON j2, J3 RCA, J4 RCA, J5 RCA, X1 STEREOJACK

Commit message: various fixes
Parts:
- removed C7: .1uF, rcl:C025-024X044
- removed J6: (no value), SparkFun-Connectors:1X05
- removed J7: (no value), SparkFun-Connectors:1X02
- removed R12, R13, R24, R26: 20k, resistor:0204V
- removed R20-PAN1: 50k, pot:B25U
- removed R8-LV1: 100k, pot:B25U
- removed X1: STEREOJACK, audio amplifier example:STX3100
- moved C13 37.6 mm to (18.1, 21.7), turned to 270 degrees
- moved L3 36.3 mm to (20.6, 29.5), turned to 180 degrees
- moved C14 34.0 mm to (15.9, 12.7), turned to 90 degrees
- moved C12 32.9 mm to (48.1, 42.5), turned to 180 degrees
- moved IC1 31.1 mm to (34.8, 36.6), turned to 180 degrees
- moved L4 27.4 mm to (22.2, 13.8), turned to 180 degrees
- moved R33 25.7 mm to (48.1, 49.4), turned to 180 degrees
- moved R19 24.7 mm to (52.7, 52.5)
- moved R17 24.4 mm to (52.8, 67.5)
- moved C11 22.7 mm to (33.0, 59.1), turned to 270 degrees
- moved R16 22.6 mm to (53.9, 71.4)
- moved R18 22.5 mm to (53.9, 56.2)
- moved D1 22.1 mm to (47.0, 20.6)
- moved R15 21.9 mm to (52.2, 80.8)
- moved R14 20.7 mm to (53.4, 85.0)
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Connections:
- removed net N$10: J6.5, X1.5
- removed net N$11: J6.4, X1.4
- removed net N$12: J6.3, X1.3
- removed net N$13: J6.2, X1.2
- removed net N$14: J6.1, X1.1
- removed net N$30: C7.1, R8-LV1.E
- removed net N$34: C7.2, J7.2
- removed net N$38: R12.1, R13.1, R8-LV1.S
- removed net N$42: R13.2, R20-PAN1.E, R26.1
- removed net N$43: R12.2, R20-PAN1.A, R24.1
- net GND: no longer J7.1, R20-PAN1.S, R8-LV1.A
- net N$51: no longer R24.2
- net N$54: no longer R26.2
Routing:
- net +12V_FILTERED: track 0.00 -> 84.6 mm
- net -12V-FILTERED: track 0.00 -> 68.1 mm
- net N$53: track 70.0 -> 29.8 mm
- net N$56: track 91.8 -> 59.9 mm
- net N$54: track 78.6 -> 48.0 mm
- net N$38: track 21.2 -> 0.00 mm
- net +12V: track 28.6 -> 44.8 mm
- net N$14: track 16.1 -> 0.00 mm
- net -12V: track 20.5 -> 33.8 mm
- net N$41: track 21.0 -> 9.01 mm
- net N$40: track 21.1 -> 9.23 mm
- net N$39: track 20.5 -> 9.84 mm
- net N$20: track 18.8 -> 8.97 mm
- net N$27: track 18.2 -> 8.88 mm
- net N$24: track 17.4 -> 8.50 mm
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